File: kicad/_saved_matrix-clock.sch (KiCad schematic (older format))
At the start: 158 parts, among them P1 CONN_02X08, P2 CONN_01X03

Commit message: board layout
Parts:
- gave numbers to parts that had none: 1
Changed lines of the file:
@@
 $EndComp
 $Comp
-L C C?
+L C C12
 U 1 1 5801A712
 P 7100 5700
-F 0 "C?" H 7125 5800 50  0000 L CNN
+F 0 "C12" H 7125 5800 50  0000 L CNN
 F 1 "100n" H 7125 5600 50  0000 L CNN
 F 2 "Capacitors_SMD:C_0603_HandSoldering" H 7138 5550 50  0001 C CNN
