File: kicad/matrix-clock.kicad_pcb (KiCad board)
At the start: 4 copper layers, 255 x 80 mm, 155 parts, among them P1 CONN_02X08, P3 CONN_01X02

Commit message: board layout
Parts:
- removed P3: CONN_01X02, Pin_Headers:Pin_Header_Straight_1x02
- added C1: 100n, Capacitors_SMD:C_0603_HandSoldering, B.Cu at (216.5, 88.3)
- added C11: 100uF, Capacitors_Tantalum_SMD:TantalC_SizeX_EIA-7343, B.Cu at (206.9, 87.3)
- added P2: CONN_01X03, Pin_Headers:Pin_Header_Straight_1x03, F.Cu at (211.5, 84.3)
- added REF**: MountingHole_3.2mm_M3_ISO7380_Pad, Mounting_Holes:MountingHole_3.2mm_M3_ISO7380_Pad, F.Cu at (114.5, 117.8)
- added REF**: MountingHole_3.2mm_M3_ISO7380_Pad, Mounting_Holes:MountingHole_3.2mm_M3_ISO7380_Pad, F.Cu at (302.5, 49.8)
- added REF**: MountingHole_3.2mm_M3_ISO7380_Pad, Mounting_Holes:MountingHole_3.2mm_M3_ISO7380_Pad, F.Cu at (302.5, 117.8)
- added REF**: MountingHole_3.2mm_M3_ISO7380_Pad, Mounting_Holes:MountingHole_3.2mm_M3_ISO7380_Pad, F.Cu at (114.5, 49.8)
- added REF***: OSHW-Logo2_14.6x12mm_SilkScreen, Symbols:OSHW-Logo2_14.6x12mm_SilkScreen, F.Cu at (116.5, 101.8)
- added REF***: KiCad-Logo2_8mm_SilkScreen, Symbols:KiCad-Logo2_8mm_SilkScreen, F.Cu at (118.6, 62.1)
- C2: footprint Capacitors_ThroughHole:C_Disc_D3_P2.5 -> Capacitors_Tantalum_SMD:TantalC_SizeX_EIA-7343; moved to B.Cu
- R1, R2, R3, R4: footprint Resistors_ThroughHole:Resistor_Horizontal_RM7mm -> Resistors_SMD:R_1206_HandSoldering
- R5, R6, R7, R8: footprint Resistors_ThroughHole:Resistor_Horizontal_RM7mm -> Resistors_SMD:R_1206_HandSoldering; moved to B.Cu
- TLC1, TLC2, TLC3, TLC4: footprint Housings_DIP:DIP-28_W7.62mm -> matrixclock:TLC5940-HTSSOP-28
- TLC5, TLC6, TLC7, TLC8: footprint Housings_DIP:DIP-28_W7.62mm -> matrixclock:TLC5940-HTSSOP-28; moved to B.Cu
- moved C2 103.8 mm to (226.3, 86.1), turned to 90 degrees
- moved TLC4 39.6 mm to (132.1, 49.6), turned to 180 degrees
- moved TLC3 39.3 mm to (132.1, 69.6), turned to 180 degrees
- moved TLC2 39.0 mm to (132.1, 89.6), turned to 180 degrees
- moved TLC1 38.6 mm to (132.1, 109.6), turned to 180 degrees
- moved R6 35.2 mm to (294.4, 94.7), turned to 90 degrees
- moved R7 35.0 mm to (294.4, 74.7), turned to 90 degrees
- moved R5 34.9 mm to (294.6, 114.9), turned to 90 degrees
- moved R8 34.2 mm to (294.9, 50.2), turned to 270 degrees
- moved P1 27.7 mm to (114.9, 73.0), turned to 0 degrees
- moved C7 20.9 mm to (298.3, 112.8), turned to 270 degrees
- moved C10 20.9 mm to (298.5, 53.8), turned to 270 degrees
- moved C9 20.7 mm to (298.3, 72.4), turned to 270 degrees
- moved C8 20.7 mm to (298.3, 91.2), turned to 270 degrees
- moved TLC7 16.2 mm to (286.4, 74.0), turned to 0 degrees
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Connections:
- C10 pad 1: +3.3VP -> +3V3
- C3 pad 1: +3.3VP -> +3V3
- C4 pad 1: +3.3VP -> +3V3
- C5 pad 1: +3.3VP -> +3V3
- C6 pad 1: +3.3VP -> +3V3
- C7 pad 1: +3.3VP -> +3V3
- C8 pad 1: +3.3VP -> +3V3
- C9 pad 1: +3.3VP -> +3V3
- P1 pad 2: Net-(P1-Pad2) -> (no net)
- R2 pad 1: Net-(R2-Pad1) -> GND
- R3 pad 1: Net-(R3-Pad1) -> GND
- R4 pad 1: Net-(R4-Pad1) -> GND
- R5 pad 1: Net-(R5-Pad1) -> GND
- R6 pad 1: Net-(R6-Pad1) -> GND
- TLC1 pad 16: Net-(TLC1-Pad16) -> (no net)
- TLC1 pad 21: +3.3VP -> +3V3
- TLC2 pad 16: Net-(TLC2-Pad16) -> (no net)
- TLC2 pad 21: +3.3VP -> +3V3
- TLC3 pad 16: Net-(TLC3-Pad16) -> (no net)
- TLC3 pad 21: +3.3VP -> +3V3
- TLC4 pad 16: Net-(TLC4-Pad16) -> (no net)
- TLC4 pad 21: +3.3VP -> +3V3
- TLC5 pad 16: Net-(TLC5-Pad16) -> (no net)
- TLC5 pad 21: +3.3VP -> +3V3
- TLC6 pad 16: Net-(TLC6-Pad16) -> (no net)
- TLC6 pad 21: +3.3VP -> +3V3
- TLC7 pad 16: Net-(TLC7-Pad16) -> (no net)
- TLC7 pad 21: +3.3VP -> +3V3
- TLC8 pad 16: Net-(TLC8-Pad16) -> (no net)
- TLC8 pad 17: Net-(TLC8-Pad17) -> (no net)
- TLC8 pad 21: +3.3VP -> +3V3
Routing:
- net +3.3VP: track 0.00 -> 1389.9 mm, vias 0 -> 1
- net GND: track 0.00 -> 969.9 mm, vias 0 -> 1
- net +3V3: track 0.00 -> 371.9 mm, vias 0 -> 7
- net Net-(D127-Pad1): track 57.1 -> 3.98 mm, vias 0 -> 1
- net Net-(D111-Pad1): track 57.3 -> 4.13 mm, vias 0 -> 1
- net Net-(D95-Pad1): track 56.9 -> 3.78 mm, vias 0 -> 1
- net Net-(D79-Pad1): track 57.0 -> 4.06 mm, vias 0 -> 1
- net Net-(D110-Pad1): track 64.7 -> 13.8 mm
- net Net-(D126-Pad1): track 64.6 -> 13.9 mm
- net Net-(D94-Pad1): track 64.3 -> 14.1 mm
- net Net-(D78-Pad1): track 64.5 -> 14.4 mm
- net Net-(D109-Pad1): track 72.5 -> 22.6 mm
- net Net-(D77-Pad1): track 71.9 -> 22.7 mm
- net Net-(D125-Pad1): track 71.8 -> 22.6 mm
- net Net-(D93-Pad1): track 71.8 -> 22.7 mm
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- added copper zone on B.Cu, net GND
- removed copper zone on In1.Cu, net +3.3VP
- removed copper zone on In2.Cu, net GND
Other:
- board size 255 x 80 mm -> 200 x 80 mm
- copper layers 4 -> 2
- net class pwr1 added: clearance 0.2, trace_width 0.8, via_dia 0.6, via_drill 0.4
- rule trace_min: 0.2 -> 0.2032
- board text added: "14.10.2016"
- board text added: "BLANK"
- board text added: "DCPRG"
- board text added: "Daniel Zerlett"
- board text added: "GND"
- board text added: "GSCLK"
- board text added: "SCK"
- board text added: "SIGNALS"
- board text added: "SIN"
- board text added: "VPRG"
- board text added: "XLAT"

Commit message: layout changes
Parts:
- added REF**: via-0.6mm, matrixclock:via-0.6mm, F.Cu at (124.8, 45.8)
- added REF**: via-0.6mm, matrixclock:via-0.6mm, F.Cu at (126.3, 59.3)
- added REF**: via-0.6mm, matrixclock:via-0.6mm, F.Cu at (124.8, 65.5)
- added REF**: via-0.6mm, matrixclock:via-0.6mm, F.Cu at (124.8, 59.3)
- added REF**: via-0.6mm, matrixclock:via-0.6mm, F.Cu at (124.5, 105.5)
- added REF**: via-0.6mm, matrixclock:via-0.6mm, F.Cu at (129.5, 98.5)
- added REF**: via-0.6mm, matrixclock:via-0.6mm, F.Cu at (124.5, 98.3)
- added REF**: via-0.6mm, matrixclock:via-0.6mm, F.Cu at (117.8, 104.8)
- added REF**: via-0.6mm, matrixclock:via-0.6mm, F.Cu at (117.8, 109.8)
- added REF**: via-0.6mm, matrixclock:via-0.6mm, F.Cu at (117.8, 99.8)
- added REF**: via-0.6mm, matrixclock:via-0.6mm, F.Cu at (117.8, 95.3)
- added REF**: via-0.6mm, matrixclock:via-0.6mm, F.Cu at (118.5, 46.8)
- added REF**: via-0.6mm, matrixclock:via-0.6mm, F.Cu at (300.0, 46.3)
- added REF**: via-0.6mm, matrixclock:via-0.6mm, F.Cu at (296.8, 46.3)
- added REF**: via-0.6mm, matrixclock:via-0.6mm, F.Cu at (297.3, 60.8)
- added REF**: via-0.6mm, matrixclock:via-0.6mm, F.Cu at (298.5, 63.0)
- added REF**: via-0.6mm, matrixclock:via-0.6mm, F.Cu at (297.8, 66.3)
- added REF**: via-0.6mm, matrixclock:via-0.6mm, F.Cu at (299.3, 68.5)
- added REF**: via-0.6mm, matrixclock:via-0.6mm, F.Cu at (297.0, 68.5)
- added REF**: via-0.6mm, matrixclock:via-0.6mm, F.Cu at (295.3, 86.5)
- added REF**: via-0.6mm, matrixclock:via-0.6mm, F.Cu at (297.0, 84.8)
- added REF**: via-0.6mm, matrixclock:via-0.6mm, F.Cu at (297.0, 82.3)
- added REF**: via-0.6mm, matrixclock:via-0.6mm, F.Cu at (136.0, 56.8)
- added REF**: via-0.6mm, matrixclock:via-0.6mm, F.Cu at (295.5, 80.8)
- added REF**: via-0.6mm, matrixclock:via-0.6mm, F.Cu at (296.0, 108.5)
- added REF**: via-0.6mm, matrixclock:via-0.6mm, F.Cu at (296.0, 105.5)
- added REF**: via-0.6mm, matrixclock:via-0.6mm, F.Cu at (296.0, 98.5)
- added REF**: via-0.6mm, matrixclock:via-0.6mm, F.Cu at (295.5, 99.8)
- added REF**: via-0.6mm, matrixclock:via-0.6mm, F.Cu at (296.8, 99.8)
- added REF**: via-0.6mm, matrixclock:via-0.6mm, F.Cu at (305.8, 56.3)
- added REF**: via-0.6mm, matrixclock:via-0.6mm, F.Cu at (305.8, 61.3)
- added REF**: via-0.6mm, matrixclock:via-0.6mm, F.Cu at (305.8, 66.3)
- added REF**: via-0.6mm, matrixclock:via-0.6mm, F.Cu at (305.8, 71.3)
- added REF**: via-0.6mm, matrixclock:via-0.6mm, F.Cu at (137.0, 57.8)
- added REF**: via-0.6mm, matrixclock:via-0.6mm, F.Cu at (305.8, 76.3)
- added REF**: via-0.6mm, matrixclock:via-0.6mm, F.Cu at (305.8, 81.3)
- added REF**: via-0.6mm, matrixclock:via-0.6mm, F.Cu at (305.8, 86.3)
- added REF**: via-0.6mm, matrixclock:via-0.6mm, F.Cu at (305.8, 91.3)
- added REF**: via-0.6mm, matrixclock:via-0.6mm, F.Cu at (305.8, 96.3)
- added REF**: via-0.6mm, matrixclock:via-0.6mm, F.Cu at (305.8, 101.3)
- added REF**: via-0.6mm, matrixclock:via-0.6mm, F.Cu at (305.8, 106.3)
- added REF**: via-0.6mm, matrixclock:via-0.6mm, F.Cu at (305.8, 111.3)
- added REF**: via-0.6mm, matrixclock:via-0.6mm, F.Cu at (124.5, 85.0)
- added REF**: via-0.6mm, matrixclock:via-0.6mm, F.Cu at (124.5, 81.5)
- added REF**: via-0.6mm, matrixclock:via-0.6mm, F.Cu at (134.5, 62.0)
- added REF**: via-0.6mm, matrixclock:via-0.6mm, F.Cu at (124.5, 83.3)
- added REF**: via-0.6mm, matrixclock:via-0.6mm, F.Cu at (124.5, 79.8)
- added REF**: via-0.6mm, matrixclock:via-0.6mm, F.Cu at (124.5, 78.0)
- added REF**: via-0.6mm, matrixclock:via-0.6mm, F.Cu at (129.0, 80.8)
- added REF**: via-0.6mm, matrixclock:via-0.6mm, F.Cu at (129.0, 79.5)
- added REF**: via-0.6mm, matrixclock:via-0.6mm, F.Cu at (129.0, 78.3)
- added REF**: via-0.6mm, matrixclock:via-0.6mm, F.Cu at (111.3, 109.5)
- added REF**: via-0.6mm, matrixclock:via-0.6mm, F.Cu at (111.3, 104.5)
- added REF**: via-0.6mm, matrixclock:via-0.6mm, F.Cu at (111.3, 99.5)
- added REF**: via-0.6mm, matrixclock:via-0.6mm, F.Cu at (111.3, 94.5)
- added REF**: via-0.6mm, matrixclock:via-0.6mm, F.Cu at (137.5, 62.0)
- added REF**: via-0.6mm, matrixclock:via-0.6mm, F.Cu at (111.3, 89.5)
- added REF**: via-0.6mm, matrixclock:via-0.6mm, F.Cu at (111.3, 84.5)
- added REF**: via-0.6mm, matrixclock:via-0.6mm, F.Cu at (111.3, 79.5)
- added REF**: via-0.6mm, matrixclock:via-0.6mm, F.Cu at (111.3, 74.5)
- added REF**: via-0.6mm, matrixclock:via-0.6mm, F.Cu at (111.3, 69.5)
- added REF**: via-0.6mm, matrixclock:via-0.6mm, F.Cu at (111.3, 64.5)
- added REF**: via-0.6mm, matrixclock:via-0.6mm, F.Cu at (111.3, 59.5)
- added REF**: via-0.6mm, matrixclock:via-0.6mm, F.Cu at (111.3, 54.5)
- added REF**: via-0.6mm, matrixclock:via-0.6mm, F.Cu at (137.3, 78.3)
- added REF**: via-0.6mm, matrixclock:via-0.6mm, F.Cu at (137.3, 76.8)
- added REF**: via-0.6mm, matrixclock:via-0.6mm, F.Cu at (129.0, 63.0)
- added REF**: via-0.6mm, matrixclock:via-0.6mm, F.Cu at (137.3, 75.3)
- added REF**: via-0.6mm, matrixclock:via-0.6mm, F.Cu at (130.0, 58.3)
- added REF**: via-0.6mm, matrixclock:via-0.6mm, F.Cu at (126.3, 65.5)
- added REF***: OSHW-Logo2_14.6x12mm_SilkScreen, Symbols:OSHW-Logo2_14.6x12mm_SilkScreen, F.Cu at (123.0, 102.0)
- added REF***: OSHW-Logo2_14.6x12mm_SilkScreen, Symbols:OSHW-Logo2_14.6x12mm_SilkScreen, F.Cu at (297.3, 105.3)
- added REF***: KiCad-Logo2_8mm_SilkScreen, Symbols:KiCad-Logo2_8mm_SilkScreen, F.Cu at (313.1, 63.8)
- added REF***: OSHW-Logo2_14.6x12mm_SilkScreen, Symbols:OSHW-Logo2_14.6x12mm_SilkScreen, F.Cu at (311.0, 103.5)
- ? (x4): renamed from REF**; value MountingHole_3.2mm_M3_ISO7380_Pad -> (none)
- C10, C3, C4, C5, C6, C7, C8, C9: value 100n -> (none)
- C2: value 100uF -> 100uF TANTALUM
- P1: value CONN_02X08 -> (none)
- P2: value CONN_01X03 -> (none)
- R1, R2, R3, R4, R5, R7: value 2k -> 1.5k
- R8: value 2k -> 1,5k
Routing:
- net /DCPRG: track 391.1 -> 360.5 mm, vias 14 -> 13
- net GND: track 969.9 -> 941.3 mm
- net +3.3VP: track 1389.9 -> 1372.1 mm
- net Net-(D104-Pad1): track 22.9 -> 18.7 mm
- net Net-(TLC4-Pad17): track 211.1 -> 214.0 mm
- net +3V3: track 371.9 -> 370.7 mm
- net Net-(D88-Pad1): track 22.2 -> 23.2 mm
- net Net-(D101-Pad1): track 25.3 -> 24.6 mm
- net /XLAT: track 393.1 -> 393.9 mm
- net /BLANK: track 393.3 -> 393.9 mm
- added copper zone on F.Cu, net +3.3VP
- added copper zone on F.Cu, net GND
Other:
- net class Default: clearance 0.2 -> 0.2032
- net class gnd: clearance 0.2 -> 0.2032
- net class pwr: clearance 0.2 -> 0.2032
- net class pwr1: clearance 0.2 -> 0.2032
- rule trace_clearance: 0.2 -> 0.2032

Commit message: finalized board
Parts:
- removed the REF*** at (123.0, 102.0)
- removed the REF*** at (297.3, 105.3)
- removed the REF*** at (311.0, 103.5)
- added REF***: OSHW-Logo2_14.6x12mm_SilkScreen, Symbols:OSHW-Logo2_14.6x12mm_SilkScreen, B.Cu at (118.6, 104.8)
- P2: footprint Pin_Headers:Pin_Header_Straight_1x03 -> matrixclock:Pin_Header_Straight_1x03_fett
- REF***: moved to B.Cu
- moved REF*** 194.6 mm to (118.6, 59.0)
- moved REF*** 3.62 mm to (118.6, 104.8)
- moved REF*** 3.05 mm to (118.6, 59.0), turned to 180 degrees
Other:
- board text added: "100n"
- board text added: "100uF"
- board text added: "100uF TANTAL"
- board text added: "3.3V LED"
- board text added: "3.3V TLC"
- board text added: "LED group of TLC1"
- board text added: "LED group of TLC2"
- board text added: "LED group of TLC3"
- board text added: "LED group of TLC4"
- board text added: "LED group of TLC5"
- board text added: "LED group of TLC6"
- board text added: "LED group of TLC7"
- board text added: "LED group of TLC8"
- board text added: "matrixclock display rev1 15.10.2016"
- board text removed: "14.10.2016"

Commit message: pcb fixes
Parts:
- removed the ? at (114.5, 117.8)
- removed the ? at (302.5, 49.8)
- removed the ? at (302.5, 117.8)
- removed the ? at (114.5, 49.8)
- removed REF** (x70): via-0.6mm, matrixclock:via-0.6mm
- removed REF*** (x2): OSHW-Logo2_14.6x12mm_SilkScreen, Symbols:OSHW-Logo2_14.6x12mm_SilkScreen
- removed REF*** (x2): KiCad-Logo2_8mm_SilkScreen, Symbols:KiCad-Logo2_8mm_SilkScreen
- added ?: MountingHole_3.2mm_M3_Pad, Mounting_Holes:MountingHole_3.2mm_M3_Pad, F.Cu at (113.5, 48.8)
- added ?: MountingHole_3.2mm_M3_Pad, Mounting_Holes:MountingHole_3.2mm_M3_Pad, F.Cu at (113.5, 118.8)
- added ?: MountingHole_3.2mm_M3_Pad, Mounting_Holes:MountingHole_3.2mm_M3_Pad, F.Cu at (303.5, 118.8)
- added ?: MountingHole_3.2mm_M3_Pad, Mounting_Holes:MountingHole_3.2mm_M3_Pad, F.Cu at (303.5, 48.8)
- C10, C3, C4, C5, C6, C7, C8, C9: value (none) -> 100n
- C2: value 100uF TANTALUM -> 100uF
- P1: value (none) -> CONN_02X08; moved to B.Cu
- P2: value (none) -> CONN_01X03; footprint matrixclock:Pin_Header_Straight_1x03_fett -> Pin_Headers:Pin_Header_Straight_1x03
- R1, R2, R3, R4, R5, R7: value 1.5k -> 2k
- R8: value 1,5k -> 2k
- moved P1 17.8 mm to (114.8, 90.8)
Connections:
- C1 pad 2: GND -> Net-(C1-Pad2)
- C10 pad 2: GND -> Net-(C10-Pad2)
- C11 pad 2: GND -> Net-(C11-Pad2)
- C2 pad 2: GND -> Net-(C1-Pad2)
- C3 pad 2: GND -> Net-(C3-Pad2)
- C4 pad 2: GND -> Net-(C4-Pad2)
- C5 pad 2: GND -> Net-(C5-Pad2)
- C6 pad 2: GND -> Net-(C6-Pad2)
- C7 pad 2: GND -> Net-(C7-Pad2)
- C8 pad 2: GND -> Net-(C8-Pad2)
- C9 pad 2: GND -> Net-(C9-Pad2)
- P1 pad 10: /XLAT -> /BLANK
- P1 pad 12: /SCLK -> /DCPRG
- P1 pad 14: Net-(P1-Pad14) -> /GSCLK
- P1 pad 16: /VPRG -> Net-(P1-Pad16)
- P1 pad 2: (no net) -> /VPRG
- P1 pad 4: /GSCLK -> Net-(P1-Pad4)
- P1 pad 6: /DCPRG -> /SCLK
- P1 pad 8: /BLANK -> /XLAT
- TLC1 pad 16: (no net) -> Net-(TLC1-Pad16)
- TLC1 pad 26: Net-(P1-Pad14) -> Net-(P1-Pad4)
- TLC2 pad 16: (no net) -> Net-(TLC2-Pad16)
- TLC3 pad 16: (no net) -> Net-(TLC3-Pad16)
- TLC4 pad 16: (no net) -> Net-(TLC4-Pad16)
- TLC5 pad 16: (no net) -> Net-(TLC5-Pad16)
- TLC6 pad 16: (no net) -> Net-(TLC6-Pad16)
- TLC7 pad 16: (no net) -> Net-(TLC7-Pad16)
- TLC8 pad 16: (no net) -> Net-(TLC8-Pad16)
- TLC8 pad 17: (no net) -> Net-(TLC8-Pad17)
Routing:
- net GND: track 941.3 -> 821.1 mm
- net Net-(P1-Pad4): track 0.00 -> 38.3 mm
- net Net-(P1-Pad14): track 38.2 -> 0.00 mm
- net Net-(C1-Pad2): track 0.00 -> 8.95 mm
- net Net-(C11-Pad2): track 0.00 -> 4.22 mm
- net Net-(C6-Pad2): track 0.00 -> 4.10 mm
- net Net-(C8-Pad2): track 0.00 -> 2.45 mm
- net Net-(C7-Pad2): track 0.00 -> 2.35 mm
- net /XLAT: track 393.9 -> 395.0 mm
Other:
- board text added: "matrixclock display rev1 19.10.2016"
- board text removed: "matrixclock display rev1 15.10.2016"

Commit message: modified board
Parts:
- added REF**: via-0.6mm, matrixclock:via-0.6mm, F.Cu at (218.0, 65.6)
- added REF**: via-0.6mm, matrixclock:via-0.6mm, F.Cu at (144.1, 59.7)
- added REF**: via-0.6mm, matrixclock:via-0.6mm, F.Cu at (234.9, 79.2)
- added REF**: via-0.6mm, matrixclock:via-0.6mm, F.Cu at (233.6, 79.2)
- added REF**: via-0.6mm, matrixclock:via-0.6mm, F.Cu at (148.4, 80.4)
- added REF**: via-0.6mm, matrixclock:via-0.6mm, F.Cu at (147.2, 80.4)
- added REF**: via-0.6mm, matrixclock:via-0.6mm, F.Cu at (145.9, 80.4)
- added REF**: via-0.6mm, matrixclock:via-0.6mm, F.Cu at (144.7, 80.4)
- added REF**: via-0.6mm, matrixclock:via-0.6mm, F.Cu at (143.4, 80.4)
- added REF**: via-0.6mm, matrixclock:via-0.6mm, F.Cu at (148.4, 79.1)
- added REF**: via-0.6mm, matrixclock:via-0.6mm, F.Cu at (147.2, 79.1)
- added REF**: via-0.6mm, matrixclock:via-0.6mm, F.Cu at (145.9, 79.1)
- added REF**: via-0.6mm, matrixclock:via-0.6mm, F.Cu at (298.6, 121.9)
- added REF**: via-0.6mm, matrixclock:via-0.6mm, F.Cu at (144.7, 79.1)
- added REF**: via-0.6mm, matrixclock:via-0.6mm, F.Cu at (143.4, 79.1)
- added REF**: via-0.6mm, matrixclock:via-0.6mm, F.Cu at (158.6, 80.4)
- added REF**: via-0.6mm, matrixclock:via-0.6mm, F.Cu at (157.3, 80.4)
- added REF**: via-0.6mm, matrixclock:via-0.6mm, F.Cu at (156.1, 80.4)
- added REF**: via-0.6mm, matrixclock:via-0.6mm, F.Cu at (154.8, 80.4)
- added REF**: via-0.6mm, matrixclock:via-0.6mm, F.Cu at (153.6, 80.4)
- added REF**: via-0.6mm, matrixclock:via-0.6mm, F.Cu at (158.6, 79.1)
- added REF**: via-0.6mm, matrixclock:via-0.6mm, F.Cu at (157.3, 79.1)
- added REF**: via-0.6mm, matrixclock:via-0.6mm, F.Cu at (156.1, 79.1)
- added REF**: via-0.6mm, matrixclock:via-0.6mm, F.Cu at (296.1, 121.9)
- added REF**: via-0.6mm, matrixclock:via-0.6mm, F.Cu at (154.8, 79.1)
- added REF**: via-0.6mm, matrixclock:via-0.6mm, F.Cu at (153.6, 79.1)
- added REF**: via-0.6mm, matrixclock:via-0.6mm, F.Cu at (178.5, 75.0)
- added REF**: via-0.6mm, matrixclock:via-0.6mm, F.Cu at (174.3, 75.0)
- added REF**: via-0.6mm, matrixclock:via-0.6mm, F.Cu at (164.4, 75.2)
- added REF**: via-0.6mm, matrixclock:via-0.6mm, F.Cu at (168.6, 75.2)
- added REF**: via-0.6mm, matrixclock:via-0.6mm, F.Cu at (154.6, 75.3)
- added REF**: via-0.6mm, matrixclock:via-0.6mm, F.Cu at (158.8, 75.3)
- added REF**: via-0.6mm, matrixclock:via-0.6mm, F.Cu at (148.8, 75.4)
- added REF**: via-0.6mm, matrixclock:via-0.6mm, F.Cu at (144.6, 75.4)
- added REF**: via-0.6mm, matrixclock:via-0.6mm, F.Cu at (293.6, 121.9)
- added REF**: via-0.6mm, matrixclock:via-0.6mm, F.Cu at (137.9, 77.9)
- added REF**: via-0.6mm, matrixclock:via-0.6mm, F.Cu at (136.6, 77.9)
- added REF**: via-0.6mm, matrixclock:via-0.6mm, F.Cu at (135.4, 77.9)
- added REF**: via-0.6mm, matrixclock:via-0.6mm, F.Cu at (139.1, 77.9)
- added REF**: via-0.6mm, matrixclock:via-0.6mm, F.Cu at (137.9, 76.7)
- added REF**: via-0.6mm, matrixclock:via-0.6mm, F.Cu at (136.6, 76.7)
- added REF**: via-0.6mm, matrixclock:via-0.6mm, F.Cu at (135.4, 76.7)
- added REF**: via-0.6mm, matrixclock:via-0.6mm, F.Cu at (134.1, 76.7)
- added REF**: via-0.6mm, matrixclock:via-0.6mm, F.Cu at (137.9, 75.4)
- added REF**: via-0.6mm, matrixclock:via-0.6mm, F.Cu at (136.6, 75.4)
- added REF**: via-0.6mm, matrixclock:via-0.6mm, F.Cu at (283.4, 121.9)
- added REF**: via-0.6mm, matrixclock:via-0.6mm, F.Cu at (135.4, 75.4)
- added REF**: via-0.6mm, matrixclock:via-0.6mm, F.Cu at (134.1, 75.4)
- added REF**: via-0.6mm, matrixclock:via-0.6mm, F.Cu at (124.5, 85.8)
- added REF**: via-0.6mm, matrixclock:via-0.6mm, F.Cu at (124.5, 84.6)
- added REF**: via-0.6mm, matrixclock:via-0.6mm, F.Cu at (124.5, 83.3)
- added REF**: via-0.6mm, matrixclock:via-0.6mm, F.Cu at (124.5, 82.1)
- added REF**: via-0.6mm, matrixclock:via-0.6mm, F.Cu at (124.5, 80.8)
- added REF**: via-0.6mm, matrixclock:via-0.6mm, F.Cu at (124.5, 79.6)
- added REF**: via-0.6mm, matrixclock:via-0.6mm, F.Cu at (124.5, 78.3)
- added REF**: via-0.6mm, matrixclock:via-0.6mm, F.Cu at (131.2, 79.8)
- added REF**: via-0.6mm, matrixclock:via-0.6mm, F.Cu at (280.9, 121.9)
- added REF**: via-0.6mm, matrixclock:via-0.6mm, F.Cu at (130.0, 79.8)
- added REF**: via-0.6mm, matrixclock:via-0.6mm, F.Cu at (128.7, 79.8)
- added REF**: via-0.6mm, matrixclock:via-0.6mm, F.Cu at (131.2, 78.6)
- added REF**: via-0.6mm, matrixclock:via-0.6mm, F.Cu at (130.0, 78.6)
- added REF**: via-0.6mm, matrixclock:via-0.6mm, F.Cu at (128.7, 78.6)
- added REF**: via-0.6mm, matrixclock:via-0.6mm, F.Cu at (168.5, 80.4)
- added REF**: via-0.6mm, matrixclock:via-0.6mm, F.Cu at (167.2, 80.4)
- added REF**: via-0.6mm, matrixclock:via-0.6mm, F.Cu at (166.0, 80.4)
- added REF**: via-0.6mm, matrixclock:via-0.6mm, F.Cu at (164.8, 80.4)
- added REF**: via-0.6mm, matrixclock:via-0.6mm, F.Cu at (163.5, 80.4)
- added REF**: via-0.6mm, matrixclock:via-0.6mm, F.Cu at (278.3, 121.9)
- added REF**: via-0.6mm, matrixclock:via-0.6mm, F.Cu at (168.5, 79.1)
- added REF**: via-0.6mm, matrixclock:via-0.6mm, F.Cu at (167.2, 79.1)
- added REF**: via-0.6mm, matrixclock:via-0.6mm, F.Cu at (166.0, 79.1)
- added REF**: via-0.6mm, matrixclock:via-0.6mm, F.Cu at (164.8, 79.1)
- added REF**: via-0.6mm, matrixclock:via-0.6mm, F.Cu at (163.5, 79.1)
- added REF**: via-0.6mm, matrixclock:via-0.6mm, F.Cu at (178.3, 80.5)
- added REF**: via-0.6mm, matrixclock:via-0.6mm, F.Cu at (177.0, 80.5)
- added REF**: via-0.6mm, matrixclock:via-0.6mm, F.Cu at (175.8, 80.5)
- added REF**: via-0.6mm, matrixclock:via-0.6mm, F.Cu at (174.5, 80.5)
- added REF**: via-0.6mm, matrixclock:via-0.6mm, F.Cu at (173.3, 80.5)
- added REF**: via-0.6mm, matrixclock:via-0.6mm, F.Cu at (275.8, 121.9)
- added REF**: via-0.6mm, matrixclock:via-0.6mm, F.Cu at (178.3, 79.2)
- added REF**: via-0.6mm, matrixclock:via-0.6mm, F.Cu at (177.0, 79.2)
- added REF**: via-0.6mm, matrixclock:via-0.6mm, F.Cu at (175.8, 79.2)
- added REF**: via-0.6mm, matrixclock:via-0.6mm, F.Cu at (174.5, 79.2)
- added REF**: via-0.6mm, matrixclock:via-0.6mm, F.Cu at (173.3, 79.2)
- added REF**: via-0.6mm, matrixclock:via-0.6mm, F.Cu at (188.4, 80.5)
- added REF**: via-0.6mm, matrixclock:via-0.6mm, F.Cu at (187.2, 80.5)
- added REF**: via-0.6mm, matrixclock:via-0.6mm, F.Cu at (185.9, 80.5)
- added REF**: via-0.6mm, matrixclock:via-0.6mm, F.Cu at (184.7, 80.5)
- added REF**: via-0.6mm, matrixclock:via-0.6mm, F.Cu at (183.4, 80.5)
- added REF**: via-0.6mm, matrixclock:via-0.6mm, F.Cu at (273.2, 121.9)
- added REF**: via-0.6mm, matrixclock:via-0.6mm, F.Cu at (188.4, 79.2)
- added REF**: via-0.6mm, matrixclock:via-0.6mm, F.Cu at (187.2, 79.2)
- added REF**: via-0.6mm, matrixclock:via-0.6mm, F.Cu at (185.9, 79.2)
- added REF**: via-0.6mm, matrixclock:via-0.6mm, F.Cu at (184.7, 79.2)
- added REF**: via-0.6mm, matrixclock:via-0.6mm, F.Cu at (183.4, 79.2)
- added REF**: via-0.6mm, matrixclock:via-0.6mm, F.Cu at (198.3, 80.4)
- added REF**: via-0.6mm, matrixclock:via-0.6mm, F.Cu at (197.1, 80.4)
- added REF**: via-0.6mm, matrixclock:via-0.6mm, F.Cu at (195.8, 80.4)
- added REF**: via-0.6mm, matrixclock:via-0.6mm, F.Cu at (194.6, 80.4)
- added REF**: via-0.6mm, matrixclock:via-0.6mm, F.Cu at (193.4, 80.4)
- added REF**: via-0.6mm, matrixclock:via-0.6mm, F.Cu at (270.7, 121.9)
- added REF**: via-0.6mm, matrixclock:via-0.6mm, F.Cu at (198.3, 79.1)
- added REF**: via-0.6mm, matrixclock:via-0.6mm, F.Cu at (197.1, 79.1)
- added REF**: via-0.6mm, matrixclock:via-0.6mm, F.Cu at (195.8, 79.1)
- added REF**: via-0.6mm, matrixclock:via-0.6mm, F.Cu at (194.6, 79.1)
- added REF**: via-0.6mm, matrixclock:via-0.6mm, F.Cu at (193.4, 79.1)
- added REF**: via-0.6mm, matrixclock:via-0.6mm, F.Cu at (208.5, 80.4)
- added REF**: via-0.6mm, matrixclock:via-0.6mm, F.Cu at (207.3, 80.4)
- added REF**: via-0.6mm, matrixclock:via-0.6mm, F.Cu at (206.0, 80.4)
- added REF**: via-0.6mm, matrixclock:via-0.6mm, F.Cu at (204.8, 80.4)
- added REF**: via-0.6mm, matrixclock:via-0.6mm, F.Cu at (203.5, 80.4)
- added REF**: via-0.6mm, matrixclock:via-0.6mm, F.Cu at (208.6, 64.8)
- added REF**: via-0.6mm, matrixclock:via-0.6mm, F.Cu at (268.2, 121.9)
- added REF**: via-0.6mm, matrixclock:via-0.6mm, F.Cu at (208.5, 79.1)
- added REF**: via-0.6mm, matrixclock:via-0.6mm, F.Cu at (207.3, 79.1)
- added REF**: via-0.6mm, matrixclock:via-0.6mm, F.Cu at (206.0, 79.1)
- added REF**: via-0.6mm, matrixclock:via-0.6mm, F.Cu at (204.8, 79.1)
- added REF**: via-0.6mm, matrixclock:via-0.6mm, F.Cu at (203.5, 79.1)
- added REF**: via-0.6mm, matrixclock:via-0.6mm, F.Cu at (214.8, 79.1)
- added REF**: via-0.6mm, matrixclock:via-0.6mm, F.Cu at (214.8, 80.1)
- added REF**: via-0.6mm, matrixclock:via-0.6mm, F.Cu at (215.1, 86.1)
- added REF**: via-0.6mm, matrixclock:via-0.6mm, F.Cu at (217.9, 83.2)
- added REF**: via-0.6mm, matrixclock:via-0.6mm, F.Cu at (219.6, 85.8)
- added REF**: via-0.6mm, matrixclock:via-0.6mm, F.Cu at (265.6, 121.9)
- added REF**: via-0.6mm, matrixclock:via-0.6mm, F.Cu at (218.1, 85.8)
- added REF**: via-0.6mm, matrixclock:via-0.6mm, F.Cu at (219.3, 80.3)
- added REF**: via-0.6mm, matrixclock:via-0.6mm, F.Cu at (218.1, 80.3)
- added REF**: via-0.6mm, matrixclock:via-0.6mm, F.Cu at (213.7, 80.1)
- added REF**: via-0.6mm, matrixclock:via-0.6mm, F.Cu at (219.3, 79.2)
- added REF**: via-0.6mm, matrixclock:via-0.6mm, F.Cu at (218.1, 79.2)
- added REF**: via-0.6mm, matrixclock:via-0.6mm, F.Cu at (213.7, 79.1)
- added REF**: via-0.6mm, matrixclock:via-0.6mm, F.Cu at (218.1, 70.7)
- added REF**: via-0.6mm, matrixclock:via-0.6mm, F.Cu at (218.1, 71.9)
- added REF**: via-0.6mm, matrixclock:via-0.6mm, F.Cu at (219.4, 71.9)
- added REF**: via-0.6mm, matrixclock:via-0.6mm, F.Cu at (263.1, 121.9)
- added REF**: via-0.6mm, matrixclock:via-0.6mm, F.Cu at (218.1, 73.2)
- added REF**: via-0.6mm, matrixclock:via-0.6mm, F.Cu at (219.4, 73.2)
- added REF**: via-0.6mm, matrixclock:via-0.6mm, F.Cu at (218.1, 74.4)
- added REF**: via-0.6mm, matrixclock:via-0.6mm, F.Cu at (219.4, 74.4)
- added REF**: via-0.6mm, matrixclock:via-0.6mm, F.Cu at (218.1, 75.7)
- added REF**: via-0.6mm, matrixclock:via-0.6mm, F.Cu at (219.4, 75.7)
- added REF**: via-0.6mm, matrixclock:via-0.6mm, F.Cu at (214.9, 75.2)
- added REF**: via-0.6mm, matrixclock:via-0.6mm, F.Cu at (213.7, 75.2)
- added REF**: via-0.6mm, matrixclock:via-0.6mm, F.Cu at (214.9, 73.9)
- added REF**: via-0.6mm, matrixclock:via-0.6mm, F.Cu at (213.7, 73.9)
- added REF**: via-0.6mm, matrixclock:via-0.6mm, F.Cu at (260.5, 121.9)
- added REF**: via-0.6mm, matrixclock:via-0.6mm, F.Cu at (214.9, 72.7)
- added REF**: via-0.6mm, matrixclock:via-0.6mm, F.Cu at (213.7, 72.7)
- added REF**: via-0.6mm, matrixclock:via-0.6mm, F.Cu at (214.9, 71.4)
- added REF**: via-0.6mm, matrixclock:via-0.6mm, F.Cu at (213.7, 71.4)
- added REF**: via-0.6mm, matrixclock:via-0.6mm, F.Cu at (214.9, 70.2)
- added REF**: via-0.6mm, matrixclock:via-0.6mm, F.Cu at (213.7, 70.2)
- added REF**: via-0.6mm, matrixclock:via-0.6mm, F.Cu at (214.9, 68.9)
- added REF**: via-0.6mm, matrixclock:via-0.6mm, F.Cu at (213.7, 68.9)
- added REF**: via-0.6mm, matrixclock:via-0.6mm, F.Cu at (214.8, 95.2)
- added REF**: via-0.6mm, matrixclock:via-0.6mm, F.Cu at (213.5, 95.2)
- added REF**: via-0.6mm, matrixclock:via-0.6mm, F.Cu at (258.0, 121.9)
- added REF**: via-0.6mm, matrixclock:via-0.6mm, F.Cu at (214.8, 94.0)
- added REF**: via-0.6mm, matrixclock:via-0.6mm, F.Cu at (213.5, 94.0)
- added REF**: via-0.6mm, matrixclock:via-0.6mm, F.Cu at (214.8, 92.7)
- added REF**: via-0.6mm, matrixclock:via-0.6mm, F.Cu at (213.5, 92.7)
- added REF**: via-0.6mm, matrixclock:via-0.6mm, F.Cu at (214.8, 91.5)
- added REF**: via-0.6mm, matrixclock:via-0.6mm, F.Cu at (213.5, 91.5)
- added REF**: via-0.6mm, matrixclock:via-0.6mm, F.Cu at (214.8, 90.3)
- added REF**: via-0.6mm, matrixclock:via-0.6mm, F.Cu at (213.5, 90.3)
- added REF**: via-0.6mm, matrixclock:via-0.6mm, F.Cu at (214.8, 89.0)
- added REF**: via-0.6mm, matrixclock:via-0.6mm, F.Cu at (219.4, 95.4)
- added REF**: via-0.6mm, matrixclock:via-0.6mm, F.Cu at (255.5, 121.9)
- added REF**: via-0.6mm, matrixclock:via-0.6mm, F.Cu at (218.1, 95.4)
- added REF**: via-0.6mm, matrixclock:via-0.6mm, F.Cu at (219.4, 94.1)
- added REF**: via-0.6mm, matrixclock:via-0.6mm, F.Cu at (218.1, 94.1)
- added REF**: via-0.6mm, matrixclock:via-0.6mm, F.Cu at (219.4, 92.9)
- added REF**: via-0.6mm, matrixclock:via-0.6mm, F.Cu at (218.1, 92.9)
- added REF**: via-0.6mm, matrixclock:via-0.6mm, F.Cu at (219.4, 91.6)
- added REF**: via-0.6mm, matrixclock:via-0.6mm, F.Cu at (218.1, 91.6)
- added REF**: via-0.6mm, matrixclock:via-0.6mm, F.Cu at (219.4, 90.4)
- added REF**: via-0.6mm, matrixclock:via-0.6mm, F.Cu at (218.1, 90.4)
- added REF**: via-0.6mm, matrixclock:via-0.6mm, F.Cu at (219.4, 89.1)
- added REF**: via-0.6mm, matrixclock:via-0.6mm, F.Cu at (252.9, 121.9)
- added REF**: via-0.6mm, matrixclock:via-0.6mm, F.Cu at (218.1, 89.1)
- added REF**: via-0.6mm, matrixclock:via-0.6mm, F.Cu at (213.5, 89.0)
- added REF**: via-0.6mm, matrixclock:via-0.6mm, F.Cu at (214.7, 99.0)
- added REF**: via-0.6mm, matrixclock:via-0.6mm, F.Cu at (213.8, 99.0)
- added REF**: via-0.6mm, matrixclock:via-0.6mm, F.Cu at (218.1, 98.9)
- added REF**: via-0.6mm, matrixclock:via-0.6mm, F.Cu at (219.1, 98.9)
- added REF**: via-0.6mm, matrixclock:via-0.6mm, F.Cu at (213.4, 115.6)
- added REF**: via-0.6mm, matrixclock:via-0.6mm, F.Cu at (214.7, 115.6)
- added REF**: via-0.6mm, matrixclock:via-0.6mm, F.Cu at (218.4, 115.6)
- added REF**: via-0.6mm, matrixclock:via-0.6mm, F.Cu at (219.6, 115.6)
- added REF**: via-0.6mm, matrixclock:via-0.6mm, F.Cu at (250.4, 121.9)
- added REF**: via-0.6mm, matrixclock:via-0.6mm, F.Cu at (219.8, 119.1)
- added REF**: via-0.6mm, matrixclock:via-0.6mm, F.Cu at (218.5, 119.1)
- added REF**: via-0.6mm, matrixclock:via-0.6mm, F.Cu at (217.3, 119.1)
- added REF**: via-0.6mm, matrixclock:via-0.6mm, F.Cu at (216.0, 119.1)
- added REF**: via-0.6mm, matrixclock:via-0.6mm, F.Cu at (214.8, 119.1)
- added REF**: via-0.6mm, matrixclock:via-0.6mm, F.Cu at (213.5, 119.1)
- added REF**: via-0.6mm, matrixclock:via-0.6mm, F.Cu at (218.2, 109.3)
- added REF**: via-0.6mm, matrixclock:via-0.6mm, F.Cu at (219.1, 109.3)
- added REF**: via-0.6mm, matrixclock:via-0.6mm, F.Cu at (214.8, 109.2)
- added REF**: via-0.6mm, matrixclock:via-0.6mm, F.Cu at (213.9, 109.2)
- added REF**: via-0.6mm, matrixclock:via-0.6mm, F.Cu at (247.8, 121.9)
- added REF**: via-0.6mm, matrixclock:via-0.6mm, F.Cu at (219.4, 105.5)
- added REF**: via-0.6mm, matrixclock:via-0.6mm, F.Cu at (213.9, 105.6)
- added REF**: via-0.6mm, matrixclock:via-0.6mm, F.Cu at (214.8, 105.6)
- added REF**: via-0.6mm, matrixclock:via-0.6mm, F.Cu at (218.4, 105.5)
- added REF**: via-0.6mm, matrixclock:via-0.6mm, F.Cu at (251.4, 105.6)
- added REF**: via-0.6mm, matrixclock:via-0.6mm, F.Cu at (256.9, 107.0)
- added REF**: via-0.6mm, matrixclock:via-0.6mm, F.Cu at (255.6, 105.9)
- added REF**: via-0.6mm, matrixclock:via-0.6mm, F.Cu at (283.5, 85.6)
- added REF**: via-0.6mm, matrixclock:via-0.6mm, F.Cu at (284.8, 85.6)
- added REF**: via-0.6mm, matrixclock:via-0.6mm, F.Cu at (286.0, 85.6)
- added REF**: via-0.6mm, matrixclock:via-0.6mm, F.Cu at (245.3, 121.9)
- added REF**: via-0.6mm, matrixclock:via-0.6mm, F.Cu at (287.3, 85.6)
- added REF**: via-0.6mm, matrixclock:via-0.6mm, F.Cu at (288.5, 85.6)
- added REF**: via-0.6mm, matrixclock:via-0.6mm, F.Cu at (289.8, 85.6)
- added REF**: via-0.6mm, matrixclock:via-0.6mm, F.Cu at (291.0, 85.6)
- added REF**: via-0.6mm, matrixclock:via-0.6mm, F.Cu at (291.0, 82.0)
- added REF**: via-0.6mm, matrixclock:via-0.6mm, F.Cu at (290.6, 105.3)
- added REF**: via-0.6mm, matrixclock:via-0.6mm, F.Cu at (289.4, 105.3)
- added REF**: via-0.6mm, matrixclock:via-0.6mm, F.Cu at (288.1, 105.3)
- added REF**: via-0.6mm, matrixclock:via-0.6mm, F.Cu at (286.9, 105.3)
- added REF**: via-0.6mm, matrixclock:via-0.6mm, F.Cu at (285.6, 105.3)
- added REF**: via-0.6mm, matrixclock:via-0.6mm, F.Cu at (209.6, 63.7)
- added REF**: via-0.6mm, matrixclock:via-0.6mm, F.Cu at (242.8, 121.9)
- added REF**: via-0.6mm, matrixclock:via-0.6mm, F.Cu at (284.4, 105.3)
- added REF**: via-0.6mm, matrixclock:via-0.6mm, F.Cu at (283.1, 105.3)
- added REF**: via-0.6mm, matrixclock:via-0.6mm, F.Cu at (289.8, 82.0)
- added REF**: via-0.6mm, matrixclock:via-0.6mm, F.Cu at (286.0, 82.0)
- added REF**: via-0.6mm, matrixclock:via-0.6mm, F.Cu at (284.8, 82.0)
- added REF**: via-0.6mm, matrixclock:via-0.6mm, F.Cu at (293.2, 67.0)
- added REF**: via-0.6mm, matrixclock:via-0.6mm, F.Cu at (293.2, 65.7)
- added REF**: via-0.6mm, matrixclock:via-0.6mm, F.Cu at (293.2, 64.5)
- added REF**: via-0.6mm, matrixclock:via-0.6mm, F.Cu at (217.9, 59.0)
- added REF**: via-0.6mm, matrixclock:via-0.6mm, F.Cu at (217.9, 60.3)
- added REF**: via-0.6mm, matrixclock:via-0.6mm, F.Cu at (240.2, 121.9)
- added REF**: via-0.6mm, matrixclock:via-0.6mm, F.Cu at (217.9, 61.5)
- added REF**: via-0.6mm, matrixclock:via-0.6mm, F.Cu at (217.9, 62.8)
- added REF**: via-0.6mm, matrixclock:via-0.6mm, F.Cu at (217.9, 64.0)
- added REF**: via-0.6mm, matrixclock:via-0.6mm, F.Cu at (214.9, 64.0)
- added REF**: via-0.6mm, matrixclock:via-0.6mm, F.Cu at (214.9, 62.8)
- added REF**: via-0.6mm, matrixclock:via-0.6mm, F.Cu at (214.9, 61.5)
- added REF**: via-0.6mm, matrixclock:via-0.6mm, F.Cu at (214.9, 60.3)
- added REF**: via-0.6mm, matrixclock:via-0.6mm, F.Cu at (214.9, 59.0)
- added REF**: via-0.6mm, matrixclock:via-0.6mm, F.Cu at (218.2, 55.5)
- added REF**: via-0.6mm, matrixclock:via-0.6mm, F.Cu at (218.2, 54.3)
- added REF**: via-0.6mm, matrixclock:via-0.6mm, F.Cu at (237.7, 121.9)
- added REF**: via-0.6mm, matrixclock:via-0.6mm, F.Cu at (218.2, 53.0)
- added REF**: via-0.6mm, matrixclock:via-0.6mm, F.Cu at (218.2, 51.8)
- added REF**: via-0.6mm, matrixclock:via-0.6mm, F.Cu at (218.2, 50.5)
- added REF**: via-0.6mm, matrixclock:via-0.6mm, F.Cu at (218.2, 49.3)
- added REF**: via-0.6mm, matrixclock:via-0.6mm, F.Cu at (214.9, 49.3)
- added REF**: via-0.6mm, matrixclock:via-0.6mm, F.Cu at (214.9, 50.5)
- added REF**: via-0.6mm, matrixclock:via-0.6mm, F.Cu at (214.9, 51.8)
- added REF**: via-0.6mm, matrixclock:via-0.6mm, F.Cu at (214.9, 53.0)
- added REF**: via-0.6mm, matrixclock:via-0.6mm, F.Cu at (214.9, 54.3)
- added REF**: via-0.6mm, matrixclock:via-0.6mm, F.Cu at (214.9, 55.5)
- added REF**: via-0.6mm, matrixclock:via-0.6mm, F.Cu at (235.1, 121.9)
- added REF**: via-0.6mm, matrixclock:via-0.6mm, F.Cu at (135.8, 57.1)
- added REF**: via-0.6mm, matrixclock:via-0.6mm, F.Cu at (135.8, 58.4)
- added REF**: via-0.6mm, matrixclock:via-0.6mm, F.Cu at (137.1, 58.4)
- added REF**: via-0.6mm, matrixclock:via-0.6mm, F.Cu at (137.1, 57.1)
- added REF**: via-0.6mm, matrixclock:via-0.6mm, F.Cu at (130.1, 59.0)
- added REF**: via-0.6mm, matrixclock:via-0.6mm, F.Cu at (128.8, 59.0)
- added REF**: via-0.6mm, matrixclock:via-0.6mm, F.Cu at (131.4, 59.0)
- added REF**: via-0.6mm, matrixclock:via-0.6mm, F.Cu at (133.9, 61.6)
- added REF**: via-0.6mm, matrixclock:via-0.6mm, F.Cu at (135.2, 61.6)
- added REF**: via-0.6mm, matrixclock:via-0.6mm, F.Cu at (136.5, 61.6)
- added REF**: via-0.6mm, matrixclock:via-0.6mm, F.Cu at (232.6, 121.9)
- added REF**: via-0.6mm, matrixclock:via-0.6mm, F.Cu at (136.5, 62.8)
- added REF**: via-0.6mm, matrixclock:via-0.6mm, F.Cu at (135.2, 62.8)
- added REF**: via-0.6mm, matrixclock:via-0.6mm, F.Cu at (133.9, 62.8)
- added REF**: via-0.6mm, matrixclock:via-0.6mm, F.Cu at (130.1, 62.8)
- added REF**: via-0.6mm, matrixclock:via-0.6mm, F.Cu at (131.4, 62.8)
- added REF**: via-0.6mm, matrixclock:via-0.6mm, F.Cu at (132.7, 62.8)
- added REF**: via-0.6mm, matrixclock:via-0.6mm, F.Cu at (128.8, 62.9)
- added REF**: via-0.6mm, matrixclock:via-0.6mm, F.Cu at (132.7, 60.3)
- added REF**: via-0.6mm, matrixclock:via-0.6mm, F.Cu at (132.7, 61.6)
- added REF**: via-0.6mm, matrixclock:via-0.6mm, F.Cu at (131.4, 61.6)
- added REF**: via-0.6mm, matrixclock:via-0.6mm, F.Cu at (230.1, 121.9)
- added REF**: via-0.6mm, matrixclock:via-0.6mm, F.Cu at (131.4, 60.3)
- added REF**: via-0.6mm, matrixclock:via-0.6mm, F.Cu at (128.8, 60.3)
- added REF**: via-0.6mm, matrixclock:via-0.6mm, F.Cu at (128.8, 61.6)
- added REF**: via-0.6mm, matrixclock:via-0.6mm, F.Cu at (130.1, 61.6)
- added REF**: via-0.6mm, matrixclock:via-0.6mm, F.Cu at (130.1, 60.3)
- added REF**: via-0.6mm, matrixclock:via-0.6mm, F.Cu at (126.3, 59.0)
- added REF**: via-0.6mm, matrixclock:via-0.6mm, F.Cu at (126.3, 60.3)
- added REF**: via-0.6mm, matrixclock:via-0.6mm, F.Cu at (126.3, 61.5)
- added REF**: via-0.6mm, matrixclock:via-0.6mm, F.Cu at (126.3, 62.8)
- added REF**: via-0.6mm, matrixclock:via-0.6mm, F.Cu at (126.3, 64.0)
- added REF**: via-0.6mm, matrixclock:via-0.6mm, F.Cu at (227.5, 121.9)
- added REF**: via-0.6mm, matrixclock:via-0.6mm, F.Cu at (126.3, 65.3)
- added REF**: via-0.6mm, matrixclock:via-0.6mm, F.Cu at (125.0, 65.3)
- added REF**: via-0.6mm, matrixclock:via-0.6mm, F.Cu at (125.0, 64.0)
- added REF**: via-0.6mm, matrixclock:via-0.6mm, F.Cu at (125.0, 62.8)
- added REF**: via-0.6mm, matrixclock:via-0.6mm, F.Cu at (125.0, 61.5)
- added REF**: via-0.6mm, matrixclock:via-0.6mm, F.Cu at (125.0, 60.3)
- added REF**: via-0.6mm, matrixclock:via-0.6mm, F.Cu at (125.0, 59.0)
- added REF**: via-0.6mm, matrixclock:via-0.6mm, F.Cu at (283.5, 82.0)
- added REF**: via-0.6mm, matrixclock:via-0.6mm, F.Cu at (225.0, 121.9)
- added REF**: via-0.6mm, matrixclock:via-0.6mm, F.Cu at (222.4, 121.9)
- added REF**: via-0.6mm, matrixclock:via-0.6mm, F.Cu at (219.9, 121.9)
- added REF**: via-0.6mm, matrixclock:via-0.6mm, F.Cu at (207.6, 63.7)
- added REF**: via-0.6mm, matrixclock:via-0.6mm, F.Cu at (217.4, 121.9)
- added REF**: via-0.6mm, matrixclock:via-0.6mm, F.Cu at (214.8, 121.9)
- added REF**: via-0.6mm, matrixclock:via-0.6mm, F.Cu at (212.3, 121.9)
- added REF**: via-0.6mm, matrixclock:via-0.6mm, F.Cu at (209.7, 121.9)
- added REF**: via-0.6mm, matrixclock:via-0.6mm, F.Cu at (207.2, 121.9)
- added REF**: via-0.6mm, matrixclock:via-0.6mm, F.Cu at (204.7, 121.9)
- added REF**: via-0.6mm, matrixclock:via-0.6mm, F.Cu at (202.1, 121.9)
- added REF**: via-0.6mm, matrixclock:via-0.6mm, F.Cu at (199.6, 121.9)
- added REF**: via-0.6mm, matrixclock:via-0.6mm, F.Cu at (197.0, 121.9)
- added REF**: via-0.6mm, matrixclock:via-0.6mm, F.Cu at (194.5, 121.9)
- added REF**: via-0.6mm, matrixclock:via-0.6mm, F.Cu at (210.8, 64.5)
- added REF**: via-0.6mm, matrixclock:via-0.6mm, F.Cu at (192.0, 121.9)
- added REF**: via-0.6mm, matrixclock:via-0.6mm, F.Cu at (189.4, 121.9)
- added REF**: via-0.6mm, matrixclock:via-0.6mm, F.Cu at (186.9, 121.9)
- added REF**: via-0.6mm, matrixclock:via-0.6mm, F.Cu at (184.3, 121.9)
- added REF**: via-0.6mm, matrixclock:via-0.6mm, F.Cu at (181.8, 121.9)
- added REF**: via-0.6mm, matrixclock:via-0.6mm, F.Cu at (179.3, 121.9)
- added REF**: via-0.6mm, matrixclock:via-0.6mm, F.Cu at (176.7, 121.9)
- added REF**: via-0.6mm, matrixclock:via-0.6mm, F.Cu at (174.2, 121.9)
- added REF**: via-0.6mm, matrixclock:via-0.6mm, F.Cu at (171.6, 121.9)
- added REF**: via-0.6mm, matrixclock:via-0.6mm, F.Cu at (169.1, 121.9)
- added REF**: via-0.6mm, matrixclock:via-0.6mm, F.Cu at (209.6, 65.7)
- added REF**: via-0.6mm, matrixclock:via-0.6mm, F.Cu at (166.6, 121.9)
- added REF**: via-0.6mm, matrixclock:via-0.6mm, F.Cu at (164.0, 121.9)
- added REF**: via-0.6mm, matrixclock:via-0.6mm, F.Cu at (161.5, 121.9)
- added REF**: via-0.6mm, matrixclock:via-0.6mm, F.Cu at (158.9, 121.9)
- added REF**: via-0.6mm, matrixclock:via-0.6mm, F.Cu at (156.4, 121.9)
- added REF**: via-0.6mm, matrixclock:via-0.6mm, F.Cu at (153.9, 121.9)
- added REF**: via-0.6mm, matrixclock:via-0.6mm, F.Cu at (151.3, 121.9)
- added REF**: via-0.6mm, matrixclock:via-0.6mm, F.Cu at (148.8, 121.9)
- added REF**: via-0.6mm, matrixclock:via-0.6mm, F.Cu at (146.2, 121.9)
- added REF**: via-0.6mm, matrixclock:via-0.6mm, F.Cu at (143.7, 121.9)
- added REF**: via-0.6mm, matrixclock:via-0.6mm, F.Cu at (212.6, 65.8)
- added REF**: via-0.6mm, matrixclock:via-0.6mm, F.Cu at (141.2, 121.9)
- added REF**: via-0.6mm, matrixclock:via-0.6mm, F.Cu at (138.6, 121.9)
- added REF**: via-0.6mm, matrixclock:via-0.6mm, F.Cu at (136.1, 121.9)
- added REF**: via-0.6mm, matrixclock:via-0.6mm, F.Cu at (133.5, 121.9)
- added REF**: via-0.6mm, matrixclock:via-0.6mm, F.Cu at (131.0, 121.9)
- added REF**: via-0.6mm, matrixclock:via-0.6mm, F.Cu at (128.5, 121.9)
- added REF**: via-0.6mm, matrixclock:via-0.6mm, F.Cu at (125.9, 121.9)
- added REF**: via-0.6mm, matrixclock:via-0.6mm, F.Cu at (123.4, 121.9)
- added REF**: via-0.6mm, matrixclock:via-0.6mm, F.Cu at (120.8, 121.9)
- added REF**: via-0.6mm, matrixclock:via-0.6mm, F.Cu at (118.3, 121.9)
- added REF**: via-0.6mm, matrixclock:via-0.6mm, F.Cu at (145.7, 61.5)
- added REF**: via-0.6mm, matrixclock:via-0.6mm, F.Cu at (274.7, 114.2)
- added REF**: via-0.6mm, matrixclock:via-0.6mm, F.Cu at (273.5, 114.2)
- added REF**: via-0.6mm, matrixclock:via-0.6mm, F.Cu at (272.2, 114.2)
- added REF**: via-0.6mm, matrixclock:via-0.6mm, F.Cu at (271.0, 114.2)
- added REF**: via-0.6mm, matrixclock:via-0.6mm, F.Cu at (269.8, 114.2)
- added REF**: via-0.6mm, matrixclock:via-0.6mm, F.Cu at (268.5, 114.2)
- added REF**: via-0.6mm, matrixclock:via-0.6mm, F.Cu at (267.3, 114.2)
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Connections:
- C1 pad 2: Net-(C1-Pad2) -> GND
- C10 pad 2: Net-(C10-Pad2) -> GND
- C11 pad 2: Net-(C11-Pad2) -> GND
- C2 pad 2: Net-(C1-Pad2) -> GND
- C3 pad 2: Net-(C3-Pad2) -> GND
- C4 pad 2: Net-(C4-Pad2) -> GND
- C5 pad 2: Net-(C5-Pad2) -> GND
- C6 pad 2: Net-(C6-Pad2) -> GND
- C7 pad 2: Net-(C7-Pad2) -> GND
- C8 pad 2: Net-(C8-Pad2) -> GND
- C9 pad 2: Net-(C9-Pad2) -> GND
Routing:
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- removed copper zone on F.Cu, net +3.3VP
